File: _autosave-engine-monitoring-unit.kicad_pcb (KiCad board)
At the start: 4 copper layers, 70 x 50 mm, 60 parts, among them J1 SW Debug, J2 Supply, J3 Oil Temperature, J4 Air Temperature, J5 Wheel Speed, J6 Inductive Sensor Wire, Q1 MMBT3904, SW1 KEY, SW2 BOOT, SW3 RST, U1 LMR16006XDDCR, U2 STM32F411CEU6, Y1 HSE, Y2 LSE

Commit message: Ground Vias
Parts:
- renumbered SW3 to RESET
Changed lines of the file:
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@@
 		(descr "http://www.alps.com/prod/info/E/HTML/Tact/SurfaceMount/SKRK/SKRKAHE020.html")
 		(tags "SMD SMT button")
-		(property "Reference" "SW3"
+		(property "Reference" "RESET"
 			(at 0 -2.75 0)
 			(layer "F.SilkS")
@@
 				(font
 					(size 1 1)
-					(thickness 0.15)
+					(thickness 0.2)
+					(bold yes)
 				)
 			)
