File: engine-monitoring-unit.kicad_pcb (KiCad board)
At the start: 4 copper layers, 70 x 50 mm, 65 parts, among them J1 SW Debug, J2 Supply, J3 Oil Temperature, J4 Air Temperature, J5 Wheel Speed, J6 Inductive Sensor Wire, J7 SW Debug, Q1 MMBT3904, SW1 KEY, SW2 BOOT, SW3 RST, U1 LMR16006XDDCR, U2 STM32F411CEU6, Y1 HSE, Y2 LSE

Commit message: Modified Layout
Parts:
- moved R8 2.80 mm to (129.1, 88.9)
- moved R10 2.60 mm to (143.0, 88.9)
- moved R13 1.25 mm to (171.2, 100.3)
Routing:
- net +3.3V: track 261.5 -> 266.9 mm
- net /PA0: track 39.1 -> 39.7 mm
Other:
- board text added: "OLED"
Changed lines of the file:
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@@
 	(footprint "Resistor_SMD:R_0603_1608Metric_Pad0.98x0.95mm_HandSolder"
 		(layer "F.Cu")
-		(at 142.975 91.515)
+		(at 142.975 88.915)
 		(descr "Resistor SMD 0603 (1608 Metric), square (rectangular) end terminal, IPC-7351 nominal with elongated pad for handsoldering. (Body size source: IPC-SM-782 page 72, https://www.pcb-3d.com/wordpress/wp-content/uploads/ipc-sm-782a_amendment_1_and_2.pdf)")
 		(tags "resistor handsolder")
@@
 	(footprint "Resistor_SMD:R_0603_1608Metric_Pad0.98x0.95mm_HandSolder"
 		(layer "F.Cu")
-		(at 171.175 101.525 -90)
+		(at 171.175 100.275 -90)
 		(descr "Resistor SMD 0603 (1608 Metric), square (rectangular) end terminal, IPC-7351 nominal with elongated pad for handsoldering. (Body size source: IPC-SM-782 page 72, https://www.pcb-3d.com/wordpress/wp-content/uploads/ipc-sm-782a_amendment_1_and_2.pdf)")
 		(tags "resistor handsolder")
@@
 	(footprint "Resistor_SMD:R_0603_1608Metric_Pad0.98x0.95mm_HandSolder"
 		(layer "F.Cu")
-		(at 129.1125 91.745)
+		(at 129.1125 88.945)
 		(descr "Resistor SMD 0603 (1608 Metric), square (rectangular) end terminal, IPC-7351 nominal with elongated pad for handsoldering. (Body size source: IPC-SM-782 page 72, https://www.pcb-3d.com/wordpress/wp-content/uploads/ipc-sm-782a_amendment_1_and_2.pdf)")
 		(tags "resistor handsolder")
@@
 	)
 	(gr_text "3.3V\n"
-		(at 166.5 105.25 0)
+		(at 167 105.5 0)
 		(layer "F.SilkS")
 		(effects
 			(font
 				(size 1 1)
-				(thickness 0.1)
+				(thickness 0.2)
+				(bold yes)
 			)
 			(justify left bottom)
@@
 	)
 	(gr_text "SDA\n"
-		(at 166.75 107.75 0)
+		(at 167 107.75 0)
 		(layer "F.SilkS")
 		(effects
 			(font
 				(size 1 1)
-				(thickness 0.1)
+				(thickness 0.2)
+				(bold yes)
 			)
 			(justify left bottom)
@@
 			(font
 				(size 1 1)
-				(thickness 0.1)
+				(thickness 0.2)
+				(bold yes)
 			)
 			(justify left bottom)
@@
 			(font
 				(size 1 1)
-				(thickness 0.1)
+				(thickness 0.2)
+				(bold yes)
 			)
 			(justify left bottom)
 		)
 	)
-	(gr_text "SWCLK\n"
-		(at 171 122.75 0)
+	(gr_text "OLED\n"
+		(at 169.35 103.7 0)
 		(layer "F.SilkS")
 		(effects
 			(font
 				(size 1 1)
-				(thickness 0.1)
+				(thickness 0.2)
+				(bold yes)
 			)
 			(justify left bottom)
 		)
 	)
-	(gr_text "SWDIO\n"
-		(at 171.25 120.25 0)
+	(gr_text "SWD"
+		(at 169.65 115.45 0)
 		(layer "F.SilkS")
 		(effects
 			(font
 				(size 1 1)
-				(thickness 0.1)
+				(thickness 0.2)
+				(bold yes)
 			)
 			(justify left bottom)
 		)
 	)
-	(gr_text "3.3V\n"
-		(at 172.5 117.75 0)
+	(gr_text "SWCLK\n"
+		(at 171 122.75 0)
 		(layer "F.SilkS")
 		(effects
 			(font
 				(size 1 1)
-				(thickness 0.1)
+				(thickness 0.2)
+				(bold yes)
 			)
 			(justify left bottom)
 		)
 	)
-	(gr_text "GND\n"
-		(at 172.75 125.25 0)
+	(gr_text "SWDIO\n"
+		(at 171.25 120.25 0)
 		(layer "F.SilkS")
 		(effects
 			(font
 				(size 1 1)
-				(thickness 0.1)
+				(thickness 0.2)
+				(bold yes)
 			)
 			(justify left bottom)
 		)
 	)
-	(gr_text "SWD"
-		(at 170.25 122.75 90)
+	(gr_text "3.3V\n"
+		(at 172.5 117.75 0)
+		(layer "F.SilkS")
+		(effects
+			(font
+				(size 1 1)
+				(thickness 0.2)
+				(bold yes)
+			)
+			(justify left bottom)
+		)
+	)
+	(gr_text "GND\n"
+		(at 172.75 125.25 0)
 		(layer "F.SilkS")
 		(effects
@@
 	)
 	(segment
-		(start 142.0625 91.515)
-		(end 142.0625 93.4375)
+		(start 127.75 93.25)
+		(end 128.2 92.8)
 		(width 0.25)
 		(layer "F.Cu")
@@
 	)
 	(segment
+		(start 142.0625 93.4375)
+		(end 142.0625 88.915)
+		(width 0.25)
+		(layer "F.Cu")
+		(net "+3.3V")
+	)
+	(segment
 		(start 161.5 117.75)
 		(end 159.25 117.75)
@@
 	)
 	(segment
-		(start 128.2 91.745)
-		(end 128.2 92.8)
-		(width 0.25)
-		(layer "F.Cu")
-		(net "+3.3V")
-	)
-	(segment
 		(start 125.4375 96.015)
 		(end 129.006 96.015)
@@
 	)
 	(segment
-		(start 171.175 100.6125)
-		(end 166.6125 100.6125)
-		(width 0.25)
-		(layer "F.Cu")
-		(net "+3.3V")
-	)
-	(segment
 		(start 144.8125 108.4375)
 		(end 145.73 108.4375)
@@
 	)
 	(segment
-		(start 166.5 105.25)
-		(end 166.5 111)
+		(start 171.175 99.3625)
+		(end 166.6125 99.3625)
+		(width 0.25)
+		(layer "F.Cu")
+		(net "+3.3V")
+	)
+	(segment
+		(start 166.5 96)
+		(end 166.5 99.25)
 		(width 0.6)
 		(layer "F.Cu")
@@
 	)
 	(segment
-		(start 128.2 92.8)
-		(end 127.75 93.25)
-		(width 0.25)
+		(start 166.5 105.25)
+		(end 166.5 111)
+		(width 0.6)
 		(layer "F.Cu")
 		(net "+3.3V")
@@
 	)
 	(segment
+		(start 128.2 92.8)
+		(end 128.2 88.945)
+		(width 0.25)
+		(layer "F.Cu")
+		(net "+3.3V")
+	)
+	(segment
 		(start 145 117.75)
 		(end 145 111.75)
@@
 	)
 	(segment
-		(start 166.5 96)
+		(start 166.5 99.25)
 		(end 166.5 104)
 		(width 0.6)
@@
 	)
 	(segment
+		(start 173.3425 102.3425)
+		(end 174.285 102.3425)
+		(width 0.25)
+		(layer "F.Cu")
+		(net "/PA0")
+	)
+	(segment
 		(start 147.25 108.5)
 		(end 147.885 107.865)
@@
 	)
 	(segment
+		(start 172.1875 101.1875)
+		(end 173.3425 102.3425)
+		(width 0.25)
+		(layer "F.Cu")
+		(net "/PA0")
+	)
+	(segment
 		(start 147.885 107.865)
 		(end 148.5325 107.865)
@@
 	)
 	(segment
-		(start 147.25 109.5)
-		(end 147.25 108.5)
+		(start 171.175 101.1875)
+		(end 172.1875 101.1875)
 		(width 0.25)
 		(layer "F.Cu")
@@
 	)
 	(segment
-		(start 175.5 102.25)
-		(end 175.4075 102.3425)
-		(width 0.3)
+		(start 147.25 109.5)
+		(end 147.25 108.5)
+		(width 0.25)
 		(layer "F.Cu")
 		(net "/PA0")
 	)
 	(segment
-		(start 171.175 102.4375)
-		(end 174.19 102.4375)
+		(start 175.5 102.25)
+		(end 175.4075 102.3425)
 		(width 0.3)
 		(layer "F.Cu")
@@
 	)
 	(segment
-		(start 145.235 91.515)
-		(end 143.8875 91.515)
+		(start 143.8875 86.0825)
+		(end 144.025 85.945)
 		(width 0.25)
 		(layer "F.Cu")
@@
 	)
 	(segment
-		(start 143.8875 91.515)
-		(end 143.8875 86.0825)
-		(width 0.25)
-		(layer "F.Cu")
-		(net "/PA3")
-	)
-	(segment
 		(start 150.975 110.725)
 		(end 150.75 110.5)
@@
 	)
 	(segment
-		(start 149.70026 110.5)
-		(end 150.75 110.5)
+		(start 143.8875 91.515)
+		(end 143.8875 86.0825)
 		(width 0.25)
 		(layer "F.Cu")
@@
 	)
 	(segment
-		(start 149.23 109.5425)
-		(end 149.23 110.02974)
+		(start 149.70026 110.5)
+		(end 150.75 110.5)
 		(width 0.25)
 		(layer "F.Cu")
@@
 	)
 	(segment
-		(start 145.735 92.015)
-		(end 145.235 91.515)
+		(start 149.23 109.5425)
+		(end 149.23 110.02974)
 		(width 0.25)
 		(layer "F.Cu")
@@
 	)
 	(segment
-		(start 143.8875 86.0825)
-		(end 144.025 85.945)
-		(width 0.25)
-		(layer "F.Cu")
-		(net "/PA3")
-	)
-	(segment
 		(start 149.9875 111.2625)
 		(end 149.75 111.5)
@@
 	)
 	(via
-		(at 145.735 92.015)
+		(at 143.8875 91.515)
 		(size 0.6)
 		(drill 0.3)
@@
 	)
 	(segment
+		(start 165.25 106.75)
+		(end 165.25 107.75)
+		(width 0.25)
+		(layer "B.Cu")
+		(net "/PA3")
+	)
+	(segment
 		(start 161.7 110.8)
 		(end 157 115.5)
@@
 	)
 	(segment
-		(start 157 115.5)
-		(end 149.75 115.5)
+		(start 162.75 95.5)
+		(end 164.75 97.5)
 		(width 0.25)
 		(layer "B.Cu")
@@
 	)
 	(segment
-		(start 145.735 92.015)
-		(end 149.22 95.5)
+		(start 157 115.5)
+		(end 149.75 115.5)
 		(width 0.25)
 		(layer "B.Cu")
@@
 	)
 	(segment
-		(start 164.75 97.5)
-		(end 164.75 106.25)
+		(start 164.75 106.25)
+		(end 165.25 106.75)
 		(width 0.25)
 		(layer "B.Cu")
@@
 	)
 	(segment
-		(start 165.25 106.75)
-		(end 164.75 106.25)
+		(start 149.22 95.5)
+		(end 162.75 95.5)
 		(width 0.25)
 		(layer "B.Cu")
@@
 	)
 	(segment
-		(start 162.75 95.5)
-		(end 164.75 97.5)
+		(start 145.235 91.515)
+		(end 149.22 95.5)
 		(width 0.25)
 		(layer "B.Cu")
@@
 	)
 	(segment
-		(start 149.22 95.5)
-		(end 162.75 95.5)
+		(start 143.8875 91.515)
+		(end 145.235 91.515)
 		(width 0.25)
 		(layer "B.Cu")
@@
 	)
 	(segment
-		(start 165.25 107.75)
-		(end 165.25 106.75)
+		(start 164.75 97.5)
+		(end 164.75 106.25)
 		(width 0.25)
 		(layer "B.Cu")
